File: harness/kicad/v2/rp-tang-harness-v2.kicad_sch (KiCad schematic)
At the start: 36 parts, among them U1 ER_OLEDM0.91_1x-I2C, U2 RP2350-PiZero, U3 Sipeed_Tang_Nano_20K, U4 Sipeed Tang Nano 20K

Commit message: kicad v2
Parts:
- removed C3: 0.1u, Capacitor_THT:C_Disc_D5.0mm_W2.5mm_P5.00mm, symbol Device:C
- removed D1: SS14, Diode_SMD:D_SOD-123, symbol Harness:D_Schottky
- removed JP1, JP2, JP3: JP, Jumper:SolderJumper-2_P1.3mm_Open_RoundedPad1.0x1.5mm, symbol Harness:JP
- removed R1, R2, R3: 220, Resistor_THT:R_Axial_DIN0207_L6.3mm_D2.5mm_P7.62mm_Horizontal, symbol Device:R
- removed R11, R12, R13, R14, R15: 1k, Resistor_THT:R_Axial_DIN0207_L6.3mm_D2.5mm_P7.62mm_Horizontal, symbol Device:R
- removed R16, R17, R18, R19, R20: 33R, Resistor_SMD:R_0603_1608Metric, symbol Harness:R
- removed R21, R22: 10k, Resistor_SMD:R_0603_1608Metric, symbol Harness:R
- removed RZ1: RP2040-Zero, MyLibrary:RP2040-Zero, symbol MyLibrary:RP2040-Zero
- removed U1: ER_OLEDM0.91_1x-I2C, MyLibrary:SSD1306 OLED 096 I2C, symbol Display_Graphic:ER_OLEDM0.91_1x-I2C
- removed U2: RP2350-PiZero, Connector_PinSocket_2.54mm:PinSocket_2x20_P2.54mm_Vertical, symbol Harness:RP2350_PiZero
- removed U4: Sipeed Tang Nano 20K, 0my_project:DIP-40_TangNano20K, symbol Harness:Tang_Nano_20K
- added A1: RaspberryPi_Pico, Module:RaspberryPi_Pico_Common_Unspecified, symbol MCU_Module:RaspberryPi_Pico
- added C4: 0.1u, Capacitor_THT:C_Disc_D5.0mm_W2.5mm_P5.00mm, symbol Device:C
- added JP1, JP2: Jumper_2_Bridged, Connector_PinHeader_2.54mm:PinHeader_1x02_P2.54mm_Vertical, symbol Jumper:Jumper_2_Bridged
- R10, R9: value 1k -> 4.7k
- R4: value 220 -> 33
- R5, R6, R7, R8: value 1k -> 33
Connections:
- net ERROR is gone; now on net HSTX_CLK: R8.2
- net IRQ_N is gone; now on net HSTX_D1: R5.2
- net LED0 is gone; now on net CS: R9.1
- net LED1 is gone; now on net RESET: R10.1
- net RESET_N is gone; now on net CS: U3.28 (86_IOT4A)
- net +3V3: now also A1.36 (3V3), C4.1
- net CIPO: now also U3.3 (75_IOT34A), A1.11 (GPIO8)
- net COPI: now also U3.17 (19_IOL51A); no longer U3.2 (74_IOT34B)
- net CS: now also A1.12 (GPIO9)
- net GND: now also R10.2, R9.2, A1.13 (GND), A1.18 (GND), A1.23 (GND), A1.28 (GND), A1.3 (GND), A1.33 (AGND), A1.38 (GND), A1.8 (GND), C4.2
- net HEARTBEAT: now also A1.10 (GPIO7), JP2.1 (A); no longer R7.2
- net HEARTBEAT_T: now also U3.6 (15_IOL46A), JP2.2 (B)
- net HSTX_CLK: now also U3.37 (80_IOT27A)
- net HSTX_CLK_P: now also R8.1, A1.21 (GPIO16)
- net HSTX_D0: now also R4.2, U3.23 (71_IOT44A)
- net HSTX_D0_P: now also R4.1, A1.16 (GPIO12)
- net HSTX_D1: now also U3.24 (72_IOT40B)
- net HSTX_D1_P: now also R5.1, A1.17 (GPIO13)
- net HSTX_D2: now also R6.2, U3.1 (73_IOT40A)
- net HSTX_D2_P: now also R6.1, A1.19 (GPIO14)
- net HSTX_D3: now also R7.2, U3.2 (74_IOT34B)
- net HSTX_D3_P: now also R7.1, A1.20 (GPIO15)
- net IRQ: now also U3.4 (85_IOT4B), A1.26 (GPIO20)
- net RESET: now also U3.27 (79_IOT27B), A1.27 (GPIO21)
- net SCK: now also U3.16 (20_IOL51B), A1.14 (GPIO10); no longer U3.1 (73_IOT40A)
- net VSYNC: now also A1.29 (GPIO22), JP1.1 (A); no longer R6.2
- net VSYNC_T: now also U3.7 (16_IOL47B), JP1.2 (B)
- net at U3.31 (48_IOR49B): no longer R8.1
- net at U3.35 (41_IOB43A): no longer R7.1
- net at U3.36 (42_IOB42B): no longer R6.1
- removed net CS_N: R4.1, U3.24 (72_IOT40B)
- no-connect marks 66 -> 44
Other:
- note removed: "JP1 + D1: Tang Nano の 5V から PiZero のヘッダ 5V へ (逆流防止)。ヘッダ 5V が VBUS か VSYS かを確認するまで JP1 は開けておき、USB を 2 本挿す。3V3 同士はつながない"
- note removed: "RP2350-PiZero - Tang Nano 20K harness v2: HSTX x4 + CLK, SPI1, IRQ/READY, VSYNC, HEARTBEAT, RESET. LCD (40pin RGB), I2S, HDMI, PIO-USB (GPIO6/7) のピンは使わない"
- moved on the sheet: U3
