File: harness/kicad/v2/rp-tang-harness-v2.kicad_sch (KiCad schematic)
At the start: 16 parts, among them U3 Sipeed_Tang_Nano_20K

Commit message: harness v2: connect COPI and Tang GND pin 26, sync docs with board
- Schematic/PCB: wire Pico pin 15 (GP11, SPI1 TX) to COPI (FPGA 19),
  tie Tang pin 26 to GND
- HARNESS2.md / pins_v2.json: new schematic path, reference designators
  (series R4-R8, pull-downs R9/R10, JP1 = VSYNC, JP2 = HEARTBEAT),
  drop the optional 5V line (JP1 + SS14) that v2 removed

Co-Authored-By: Claude Opus 5.5 (1M context) <noreply@anthropic.com>
Connections:
- net COPI: now also A1.15 (GPIO11)
- net GND: now also U3.26 (GND)
- no-connect marks 44 -> 42
Changed lines of the file:
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@@
-	)
-	(no_connect
-		(at 171.45 67.31)
 	)
 	(no_connect
@@
 	)
 	(no_connect
-		(at 34.29 83.82)
-	)
-	(no_connect
 		(at 57.15 33.02)
 	)
@@
 	(wire
 		(pts
+			(xy 171.45 67.31) (xy 185.42 67.31)
+		)
+		(stroke
+			(width 0)
+			(type default)
+		)
+	)
+	(wire
+		(pts
 			(xy 121.92 72.39) (xy 135.89 72.39)
 		)
@@
 		(pts
 			(xy 21.59 88.9) (xy 34.29 88.9)
+		)
+		(stroke
+			(width 0)
+			(type default)
+		)
+	)
+	(wire
+		(pts
+			(xy 21.59 83.82) (xy 34.29 83.82)
 		)
 		(stroke
@@
 	(label "RESET"
 		(at 30.48 148.59 0)
+		(effects
+			(font
+				(size 1.27 1.27)
+			)
+			(justify left bottom)
+		)
+	)
+	(label "COPI"
+		(at 21.59 83.82 0)
 		(effects
 			(font
@@
 					(unit 1)
 				)
+			)
+		)
+	)
+	(symbol
+		(lib_id "power:GND")
+		(at 185.42 67.31 0)
+		(unit 1)
+		(body_style 1)
+		(exclude_from_sim no)
+		(in_bom yes)
+		(on_board yes)
+		(in_pos_files yes)
+		(dnp no)
+		(fields_autoplaced yes)
+		(property "Reference" "#PWR08"
+			(at 185.42 73.66 0)
+			(hide yes)
+			(show_name no)
+			(do_not_autoplace no)
+			(effects
+				(font
+					(size 1.27 1.27)
+				)
+			)
+		)
+		(property "Value" "GND"
+			(at 185.42 72.39 0)
+			(show_name no)
+			(do_not_autoplace no)
+			(effects
+				(font
+					(size 1.27 1.27)
+				)
+			)
+		)
+		(property "Footprint" ""
+			(at 185.42 67.31 0)
+			(hide yes)
+			(show_name no)
+			(do_not_autoplace no)
+			(effects
+				(font
+					(size 1.27 1.27)
+				)
+			)
+		)
+		(property "Datasheet" ""
+			(at 185.42 67.31 0)
+			(hide yes)
+			(show_name no)
+			(do_not_autoplace no)
+			(effects
+				(font
+					(size 1.27 1.27)
+				)
+			)
+		)
+		(property "Description" "Power symbol creates a global label with name \"GND\" , ground"
+			(at 185.42 67.31 0)
+			(hide yes)
+			(show_name no)
+			(do_not_autoplace no)
+			(effects
+				(font
+					(size 1.27 1.27)
+				)
+			)
+		)
+		(pin "1"
+		)
+		(instances
+			(project "rp-tang-harness-v2"
+				(path "/2cf01f59-cf54-439e-881f-c06c5145d63c"
+					(reference "#PWR08")
+					(unit 1)
+				)

Commit message: harness v2: move VSYNC to DDC_CLK (52), drop HEARTBEAT and jumpers
- KiCad: VSYNC Pico pin 29 -> Tang 52 (HDMI DDC_CLK, 2.2k pull-up to 3.3V),
  direct trace. JP1/JP2 and the HEARTBEAT line removed
- HARNESS2.md / pins_v2.json: 12 signals. HEARTBEAT only mirrored VSYNC
  (both stop in reset), so ready is judged from VSYNC edges. 15-18 are free
  for LCD_INIT; 76 stays unused (BL616 JTAG MOSI)

Co-Authored-By: Claude Opus 5.5 (1M context) <noreply@anthropic.com>
Parts:
- removed JP1, JP2: Jumper_2_Bridged, Connector_PinHeader_2.54mm:PinHeader_1x02_P2.54mm_Vertical, symbol Jumper:Jumper_2_Bridged
Connections:
- net VSYNC: now also U3.21 (52_IOR39A)
- net VSYNC_T: no longer names the net of U3.7 (16_IOL47B)
Other:
- note removed: "JP2, JP3: FPGA 15/16 は LCD の XR/YD (LCD_INIT0/1) と共有。それを使うパネルのときだけ開ける (既定は閉)"
