File: harness/kicad/v2/rp-tang-harness-v2.kicad_sch (KiCad schematic)
At the start: 14 parts, among them U3 Sipeed_Tang_Nano_20K

Commit message: cleanup
Connections:
- net HEARTBEAT: no longer names the net of A1.10 (GPIO7)
- net HEARTBEAT_T: no longer names the net of U3.6 (15_IOL46A)
- no-connect marks 42 -> 44
Changed lines of the file:
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@@
+	)
+	(no_connect
+		(at 135.89 44.45)
 	)
 	(no_connect
@@
 	)
 	(no_connect
+		(at 34.29 73.66)
+	)
+	(no_connect
 		(at 171.45 31.75)
 	)
@@
 	(wire
 		(pts
-			(xy 123.19 44.45) (xy 135.89 44.45)
-		)
-		(stroke
-			(width 0)
-			(type default)
-		)
-	)
-	(wire
-		(pts
 			(xy 181.61 39.37) (xy 171.45 39.37)
-		)
-		(stroke
-			(width 0)
-			(type default)
-		)
-	)
-	(wire
-		(pts
-			(xy 21.59 73.66) (xy 34.29 73.66)
 		)
 		(stroke
@@
 		)
 	)
-	(label "HEARTBEAT"
-		(at 21.59 73.66 0)
-		(effects
-			(font
-				(size 1.27 1.27)
-			)
-			(justify left bottom)
-		)
-	)
 	(label "HSTX_D3_P"
 		(at 21.59 93.98 0)
@@
 		)
 	)
-	(label "HEARTBEAT_T"
-		(at 123.19 44.45 0)
-		(effects
-			(font
-				(size 1.27 1.27)
-			)
-			(justify left bottom)
-		)
-	)
