File: harness/kicad/v2/rp-tang-harness-v2.kicad_pcb (KiCad board)
At the start: 2 copper layers, 56 x 76 mm, 23 parts, among them U1 ER_OLEDM0.91_1x-I2C, U3 Sipeed_Tang_Nano_20K

Commit message: kicad v2
Parts:
- removed C3: 0.1u, Capacitor_THT:C_Disc_D5.0mm_W2.5mm_P5.00mm
- removed R1, R2, R3: 220, Resistor_THT:R_Axial_DIN0207_L6.3mm_D2.5mm_P7.62mm_Horizontal
- removed R11, R12, R13, R14, R15: 1k, Resistor_THT:R_Axial_DIN0207_L6.3mm_D2.5mm_P7.62mm_Horizontal
- removed RZ1: RP2040-Zero, MyLibrary:RP2040-Zero
- removed U1: ER_OLEDM0.91_1x-I2C, MyLibrary:SSD1306 OLED 096 I2C
- added A1: RaspberryPi_Pico, Module:RaspberryPi_Pico_Common_Unspecified, F.Cu at (147.6, 81.3)
- added C4: 0.1u, Capacitor_THT:C_Disc_D5.0mm_W2.5mm_P5.00mm, F.Cu at (133.5, 67.6)
- added JP1: Jumper_2_Bridged, Connector_PinHeader_2.54mm:PinHeader_1x02_P2.54mm_Vertical, F.Cu at (124.4, 100.5)
- added JP2: Jumper_2_Bridged, Connector_PinHeader_2.54mm:PinHeader_1x02_P2.54mm_Vertical, F.Cu at (128.0, 100.5)
- R10, R9: value 1k -> 4.7k
- R4: value 220 -> 33
- R5, R6, R7, R8: value 1k -> 33
- moved R4 32.6 mm to (161.0, 98.0), turned to -90 degrees
- moved R10 32.3 mm to (156.4, 67.2), turned to 180 degrees
- moved R7 13.3 mm to (171.4, 98.0), turned to -90 degrees
- moved R6 8.87 mm to (167.8, 98.0), turned to -90 degrees
- moved R5 8.50 mm to (164.4, 98.0), turned to -90 degrees
- moved R8 8.04 mm to (157.6, 98.0), turned to -90 degrees
- moved R9 3.19 mm to (151.4, 95.2), turned to 180 degrees
Connections:
- R10 pad 1: /LED1 -> /RESET
- R10 pad 2: Net-(U3-16_IOL47B) -> GND
- R4 pad 1: /CS_N -> /HSTX_D0_P
- R4 pad 2: Net-(RZ1-GP5) -> /HSTX_D0
- R5 pad 1: Net-(U3-71_IOT44A) -> /HSTX_D1_P
- R5 pad 2: /IRQ_N -> /HSTX_D1
- R6 pad 1: Net-(U3-42_IOB42B) -> /HSTX_D2_P
- R6 pad 2: /VSYNC -> /HSTX_D2
- R7 pad 1: Net-(U3-41_IOB43A) -> /HSTX_D3_P
- R7 pad 2: /HEARTBEAT -> /HSTX_D3
- R8 pad 1: Net-(U3-48_IOR49B) -> /HSTX_CLK_P
- R8 pad 2: /ERROR -> /HSTX_CLK
- R9 pad 1: /LED0 -> /CS
- R9 pad 2: Net-(U3-15_IOL46A) -> GND
- U3 pad 1: /SCK -> /HSTX_D2
- U3 pad 15: Net-(U3-17_IOL49A) -> unconnected-(U3-17_IOL49A-Pad15)
- U3 pad 16: Net-(U3-20_IOL51B) -> /SCK
- U3 pad 17: Net-(U3-19_IOL51A) -> /COPI
- U3 pad 18: Net-(U3-18_IOL49B) -> unconnected-(U3-18_IOL49B-Pad18)
- U3 pad 2: /COPI -> /HSTX_D3
- U3 pad 23: Net-(U3-71_IOT44A) -> /HSTX_D0
- U3 pad 24: /CS_N -> /HSTX_D1
- U3 pad 27: unconnected-(U3-79_IOT27B-Pad27) -> /RESET
- U3 pad 28: /RESET_N -> /CS
- U3 pad 3: Net-(U3-75_IOT34A) -> /CIPO
- U3 pad 31: Net-(U3-48_IOR49B) -> unconnected-(U3-48_IOR49B-Pad31)
- U3 pad 35: Net-(U3-41_IOB43A) -> unconnected-(U3-41_IOB43A-Pad35)
- U3 pad 36: Net-(U3-42_IOB42B) -> unconnected-(U3-42_IOB42B-Pad36)
- U3 pad 37: unconnected-(U3-80_IOT27A-Pad37) -> /HSTX_CLK
- U3 pad 4: unconnected-(U3-85_IOT4B-Pad4) -> /IRQ
- U3 pad 6: Net-(U3-15_IOL46A) -> /HEARTBEAT_T
- U3 pad 7: Net-(U3-16_IOL47B) -> /VSYNC_T
Routing:
- net /COPI: track 85.3 -> 0.00 mm, vias 1 -> 0
- net /IRQ: track 0.00 -> 71.5 mm, vias 0 -> 1
- net /CIPO: track 107.3 -> 46.4 mm, vias 0 -> 1
- net /HSTX_D3: track 0.00 -> 53.5 mm
- net /CS_N: track 52.3 -> 0.00 mm, vias 1 -> 0
- net /HSTX_D2: track 0.00 -> 52.2 mm
- net +3V3: track 53.8 -> 4.86 mm, vias 1 -> 0
- net /VSYNC_T: track 0.00 -> 45.1 mm
- net /I2C_SDA: track 44.6 -> 0.00 mm
- net /HEARTBEAT_T: track 0.00 -> 43.1 mm
- net /SCK: track 86.0 -> 43.1 mm
- net /RESET: track 0.00 -> 43.0 mm, vias 0 -> 1
- net /IRQ_N: track 41.5 -> 0.00 mm
- net /HSTX_CLK_P: track 0.00 -> 40.2 mm
- net Net-(U3-20_IOL51B): track 39.3 -> 0.00 mm
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Other:
- outline, holes or cut-outs redrawn
- board text added: "rp-tang-harness v0.2 (c) 2026 Youichi Fujimoto"
- board text removed: "rp-tang-harness v0.1 (c) 2026 Youichi Fujimoto"

Commit message: wip
Routing:
- net /HEARTBEAT_T: track 43.1 -> 30.5 mm, vias 0 -> 1
- net /VSYNC_T: track 45.1 -> 34.2 mm, vias 0 -> 1
- net /VSYNC: track 47.9 -> 42.0 mm
- net /IRQ: track 71.5 -> 67.3 mm
- net /HSTX_D0_P: track 8.01 -> 7.25 mm
- net /HEARTBEAT: track 23.0 -> 22.3 mm
- net /HSTX_D2: track 52.2 -> 52.8 mm
- net /CIPO: vias 1 -> 2
- net GND: vias 3 -> 2
- net /HSTX_CLK: vias 1 -> 0
