File: harness/kicad/v2/rp-tang-harness-v2.kicad_pcb (KiCad board)
At the start: 2 copper layers, 56 x 76 mm, 16 parts, among them U3 Sipeed_Tang_Nano_20K

Commit message: harness v2: connect COPI and Tang GND pin 26, sync docs with board
- Schematic/PCB: wire Pico pin 15 (GP11, SPI1 TX) to COPI (FPGA 19),
  tie Tang pin 26 to GND
- HARNESS2.md / pins_v2.json: new schematic path, reference designators
  (series R4-R8, pull-downs R9/R10, JP1 = VSYNC, JP2 = HEARTBEAT),
  drop the optional 5V line (JP1 + SS14) that v2 removed

Co-Authored-By: Claude Opus 5.5 (1M context) <noreply@anthropic.com>
Connections:
- A1 pad 15: unconnected-(A1-GPIO11-Pad15)_1 -> /COPI
- U3 pad 26: unconnected-(U3-GND-Pad26) -> GND
Routing:
- net /COPI: track 0.00 -> 42.5 mm
- net GND: vias 2 -> 3
- net /HSTX_D1: vias 1 -> 0
Changed lines of the file:
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@@
 			(layers "F.Cu" "F.Mask")
 			(roundrect_rratio 0.5)
-			(net "unconnected-(A1-GPIO11-Pad15)")
+			(net "/COPI")
 			(pinfunction "GPIO11_15")
-			(pintype "bidirectional+no_connect")
+			(pintype "bidirectional")
 		)
 		(pad "15" thru_hole circle
@@
 			(layers "*.Cu" "*.Mask")
 			(remove_unused_layers no)
-			(net "unconnected-(A1-GPIO11-Pad15)_1")
+			(net "/COPI")
 			(pinfunction "GPIO11_15")
-			(pintype "bidirectional+no_connect")
+			(pintype "bidirectional")
 		)
 		(pad "16" smd roundrect
@@
 			(layers "*.Cu" "*.Mask")
 			(remove_unused_layers no)
-			(net "unconnected-(U3-GND-Pad26)")
+			(net "GND")
 			(pinfunction "GND_26")
-			(pintype "power_in+no_connect")
+			(pintype "power_in")
 			(thermal_bridge_angle 45)
 		)
@@
 	)
 	(via
+		(at 157.1 113.9)
+		(size 0.6)
+		(drill 0.3)
+		(layers "F.Cu" "B.Cu")
+		(free yes)
+		(net "GND")
+	)
+	(via
 		(at 145.3 120.4)
 		(size 0.6)
@@
 		(net "/HSTX_CLK")
 	)
-	(via
-		(at 166.51 108.84)
-		(size 0.6)
-		(drill 0.3)
-		(layers "F.Cu" "B.Cu")
-		(net "/HSTX_D1")
-	)
 	(segment
 		(start 164.4 105.61)
@@
 	)
 	(segment
+		(start 158.7 91.3)
+		(end 159 91)
+		(width 0.2)
+		(layer "F.Cu")
+		(net "/COPI")
+	)
+	(segment
+		(start 160.1 122.75)
+		(end 166.51 129.16)
+		(width 0.2)
+		(layer "B.Cu")
+		(net "/COPI")
+	)
+	(segment
+		(start 159.9 94.9)
+		(end 159.9 106.9)
+		(width 0.2)
+		(layer "B.Cu")
+		(net "/COPI")
+	)
+	(segment
+		(start 159 90.2)
+		(end 159 94)
+		(width 0.2)
+		(layer "B.Cu")
+		(net "/COPI")
+	)
+	(segment
+		(start 159 94)
+		(end 159.9 94.9)
+		(width 0.2)
+		(layer "B.Cu")
+		(net "/COPI")
+	)
+	(segment
+		(start 159.9 106.9)
+		(end 160.1 107.1)
+		(width 0.2)
+		(layer "B.Cu")
+		(net "/COPI")
+	)
+	(segment
+		(start 160.1 107.1)
+		(end 160.1 122.75)
+		(width 0.2)
+		(layer "B.Cu")
+		(net "/COPI")
+	)
+	(segment

Commit message: harness v2: move VSYNC to DDC_CLK (52), drop HEARTBEAT and jumpers
- KiCad: VSYNC Pico pin 29 -> Tang 52 (HDMI DDC_CLK, 2.2k pull-up to 3.3V),
  direct trace. JP1/JP2 and the HEARTBEAT line removed
- HARNESS2.md / pins_v2.json: 12 signals. HEARTBEAT only mirrored VSYNC
  (both stop in reset), so ready is judged from VSYNC edges. 15-18 are free
  for LCD_INIT; 76 stays unused (BL616 JTAG MOSI)

Co-Authored-By: Claude Opus 5.5 (1M context) <noreply@anthropic.com>
Parts:
- removed JP1, JP2: Jumper_2_Bridged, Connector_PinHeader_2.54mm:PinHeader_1x02_P2.54mm_Vertical
Connections:
- U3 pad 21: unconnected-(U3-52_IOR39A-Pad21) -> /VSYNC
- U3 pad 7: /VSYNC_T -> unconnected-(U3-16_IOL47B-Pad7)
Routing:
- net /VSYNC_T: track 34.2 -> 0.00 mm, vias 1 -> 0
- net /HEARTBEAT_T: track 30.5 -> 4.58 mm
- net /HEARTBEAT: track 22.3 -> 0.00 mm
- net unconnected-(U3-16_IOL47B-Pad7): track 0.00 -> 8.37 mm, vias 0 -> 1
- net /VSYNC: track 42.0 -> 46.5 mm, vias 0 -> 2
