File: harness/kicad/v2/rp-tang-harness-v2.kicad_pcb (KiCad board)
At the start: 2 copper layers, 56 x 76 mm, 14 parts, among them U3 Sipeed_Tang_Nano_20K

Commit message: cleanup
Connections:
- A1 pad 10: /HEARTBEAT -> unconnected-(A1-GPIO7-Pad10)_1
- U3 pad 6: /HEARTBEAT_T -> unconnected-(U3-15_IOL46A-Pad6)
Routing:
- net unconnected-(U3-15_IOL46A-Pad6): track 0.00 -> 4.58 mm, vias 0 -> 1
- net /HEARTBEAT_T: track 4.58 -> 0.00 mm, vias 1 -> 0
Changed lines of the file:
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@@
 			(layers "F.Cu" "F.Mask")
 			(roundrect_rratio 0.5)
-			(net "/HEARTBEAT")
+			(net "unconnected-(A1-GPIO7-Pad10)")
 			(pinfunction "GPIO7_10")
-			(pintype "bidirectional")
+			(pintype "bidirectional+no_connect")
 		)
 		(pad "10" thru_hole circle
@@
 			(layers "*.Cu" "*.Mask")
 			(remove_unused_layers no)
-			(net "/HEARTBEAT")
+			(net "unconnected-(A1-GPIO7-Pad10)_1")
 			(pinfunction "GPIO7_10")
-			(pintype "bidirectional")
+			(pintype "bidirectional+no_connect")
 		)
 		(pad "11" smd roundrect
@@
 			(layers "*.Cu" "*.Mask")
 			(remove_unused_layers no)
-			(net "/HEARTBEAT_T")
+			(net "unconnected-(U3-15_IOL46A-Pad6)")
 			(pinfunction "15_IOL46A_6")
-			(pintype "bidirectional")
+			(pintype "bidirectional+no_connect")
 			(thermal_bridge_angle 45)
 		)
@@
 		(net "+3V3")
 	)
-	(via
-		(at 136.4 125.5)
-		(size 0.6)
-		(drill 0.3)
-		(layers "F.Cu" "B.Cu")
-		(net "/HEARTBEAT_T")
-	)
-	(segment
-		(start 136.44 125.5)
-		(end 138.57 127.63)
-		(width 0.2)
-		(layer "B.Cu")
-		(net "/HEARTBEAT_T")
-	)
-	(segment
-		(start 138.57 127.63)
-		(end 138.57 129.16)
-		(width 0.2)
-		(layer "B.Cu")
-		(net "/HEARTBEAT_T")
-	)
-	(segment
-		(start 136.4 125.5)
-		(end 136.44 125.5)
-		(width 0.2)
-		(layer "B.Cu")
-		(net "/HEARTBEAT_T")
-	)
 	(segment
 		(start 157.6 105.6)
@@
 		(net "/HSTX_D3")
 	)
+	(via
+		(at 135.3 124.4)
+		(size 0.6)
+		(drill 0.3)
+		(layers "F.Cu" "B.Cu")
+		(net "unconnected-(U3-16_IOL47B-Pad7)")
+	)
+	(segment
+		(start 141.11 128.161471)
+		(end 141.11 129.16)
+		(width 0.2)
+		(layer "B.Cu")
+		(net "unconnected-(U3-16_IOL47B-Pad7)")
+	)
+	(segment
+		(start 135.3 124.4)
+		(end 137.348529 124.4)
+		(width 0.2)
+		(layer "B.Cu")
+		(net "unconnected-(U3-16_IOL47B-Pad7)")
+	)
+	(segment
+		(start 137.348529 124.4)
+		(end 141.11 128.161471)
+		(width 0.2)
+		(layer "B.Cu")
+		(net "unconnected-(U3-16_IOL47B-Pad7)")
+	)
 	(segment
 		(start 162.1 104.51)
@@
 	)
 	(via
-		(at 135.3 124.4)
+		(at 136.4 125.5)
 		(size 0.6)
 		(drill 0.3)
 		(layers "F.Cu" "B.Cu")
-		(net "unconnected-(U3-16_IOL47B-Pad7)")
+		(net "unconnected-(U3-15_IOL46A-Pad6)")
 	)
 	(segment
-		(start 141.11 128.161471)
-		(end 141.11 129.16)
+		(start 136.44 125.5)
+		(end 138.57 127.63)
 		(width 0.2)
 		(layer "B.Cu")
-		(net "unconnected-(U3-16_IOL47B-Pad7)")
+		(net "unconnected-(U3-15_IOL46A-Pad6)")
 	)
 	(segment
-		(start 135.3 124.4)
-		(end 137.348529 124.4)
+		(start 138.57 127.63)
+		(end 138.57 129.16)
 		(width 0.2)
 		(layer "B.Cu")
-		(net "unconnected-(U3-16_IOL47B-Pad7)")
+		(net "unconnected-(U3-15_IOL46A-Pad6)")
 	)
 	(segment
-		(start 137.348529 124.4)
-		(end 141.11 128.161471)
+		(start 136.4 125.5)
+		(end 136.44 125.5)
 		(width 0.2)
 		(layer "B.Cu")
-		(net "unconnected-(U3-16_IOL47B-Pad7)")
+		(net "unconnected-(U3-15_IOL46A-Pad6)")
 	)
 	(zone
